File: hardware/esp8266.sch (KiCad schematic (older format))
At the start: 21 parts

Commit message: Changed esp8266 chip_en
Parts:
- added C?: 100nF, symbol Device:C
- added R?: 10K, symbol Device:R
Connections:
- net labels added: CHIP_DISABLE, RX, TX
- net labels removed: CHIP_LOW_POWER
- wire segments 55 -> 59
Other:
- moved on the sheet: R?
Changed lines of the file:
@@
 L power:GND #PWR?
 U 1 1 603AB349
-P 6850 3850
-F 0 "#PWR?" H 6850 3600 50  0001 C CNN
-F 1 "GND" H 6855 3677 50  0000 C CNN
-F 2 "" H 6850 3850 50  0001 C CNN
-F 3 "" H 6850 3850 50  0001 C CNN
-	1    6850 3850
+P 7150 3850
+F 0 "#PWR?" H 7150 3600 50  0001 C CNN
+F 1 "GND" H 7155 3677 50  0000 C CNN
+F 2 "" H 7150 3850 50  0001 C CNN
+F 3 "" H 7150 3850 50  0001 C CNN
+	1    7150 3850
 	1    0    0    -1
 $EndComp
@@
 U 1 1 603AFF1C
 P 5950 3250
-F 0 "R?" V 5743 3250 50  0000 C CNN
-F 1 "10K" V 5834 3250 50  0000 C CNN
+F 0 "R?" V 5900 3100 50  0000 C CNN
+F 1 "10K" V 5950 3250 50  0000 C CNN
 F 2 "" V 5880 3250 50  0001 C CNN
 F 3 "~" H 5950 3250 50  0001 C CNN
@@
 L Device:R R?
 U 1 1 60338D72
-P 2150 6400
-F 0 "R?" H 2080 6354 50  0000 R CNN
-F 1 "10K" H 2080 6445 50  0000 R CNN
-F 2 "" V 2080 6400 50  0001 C CNN
-F 3 "~" H 2150 6400 50  0001 C CNN
-	1    2150 6400
+P 2150 6250
+F 0 "R?" H 2080 6204 50  0000 R CNN
+F 1 "10K" H 2080 6295 50  0000 R CNN
+F 2 "" V 2080 6250 50  0001 C CNN
+F 3 "~" H 2150 6250 50  0001 C CNN
+	1    2150 6250
 	-1   0    0    1
 $EndComp
@@
 L power:+3.3V #PWR?
 U 1 1 6033B326
-P 2150 6250
-F 0 "#PWR?" H 2150 6100 50  0001 C CNN
-F 1 "+3.3V" H 2165 6423 50  0000 C CNN
-F 2 "" H 2150 6250 50  0001 C CNN
-F 3 "" H 2150 6250 50  0001 C CNN
-	1    2150 6250
+P 2150 6100
+F 0 "#PWR?" H 2150 5950 50  0001 C CNN
+F 1 "+3.3V" H 2165 6273 50  0000 C CNN
+F 2 "" H 2150 6100 50  0001 C CNN
+F 3 "" H 2150 6100 50  0001 C CNN
+	1    2150 6100
 	1    0    0    -1
 $EndComp
@@
 $EndComp
 Text HLabel 1350 6750 0    50   Input ~ 0
-CHIP_LOW_POWER
+CHIP_DISABLE
 $Comp
 L Device:R R?
@@
 Wire Wire Line
 	3500 2850 3850 2850
-Text Label 2400 6550 0    50   ~ 0
+Text Label 2400 6400 0    50   ~ 0
 CHIP_PU
-Wire Wire Line
-	2400 6550 2150 6550
 $Comp
 L Device:Q_NMOS_GDS Q?
@@
 	1    0    0    -1
 $EndComp
-Connection ~ 2150 6550
+$Comp
+L Device:C C?
+U 1 1 6034AC2C
+P 1900 6400
+F 0 "C?" V 1648 6400 50  0000 C CNN
+F 1 "100nF" V 1739 6400 50  0000 C CNN
+F 2 "" H 1938 6250 50  0001 C CNN
+F 3 "~" H 1900 6400 50  0001 C CNN
+	1    1900 6400
+	0    1    1    0
+$EndComp
+$Comp
+L power:GND #PWR?
+U 1 1 6034CB2C
+P 1750 6400
+F 0 "#PWR?" H 1750 6150 50  0001 C CNN
+F 1 "GND" H 1755 6227 50  0000 C CNN
+F 2 "" H 1750 6400 50  0001 C CNN
+F 3 "" H 1750 6400 50  0001 C CNN
+	1    1750 6400
+	1    0    0    -1
+$EndComp
+Wire Wire Line
+	2150 6550 2150 6400
+Wire Wire Line
+	2400 6400 2150 6400
+Connection ~ 2150 6400
+Wire Wire Line
+	2150 6400 2050 6400
+Text HLabel 6350 3150 2    50   Output ~ 0
+TX
+Text HLabel 6350 3050 2    50   Input ~ 0
+RX
+Wire Wire Line
+	5650 3150 6350 3150
+Wire Wire Line
+	5650 3050 6350 3050
+$Comp
+L Device:R R?
+U 1 1 60357BFC
+P 7000 3850
+F 0 "R?" V 6793 3850 50  0000 C CNN
+F 1 "10K" V 6884 3850 50  0000 C CNN
+F 2 "" V 6930 3850 50  0001 C CNN
+F 3 "~" H 7000 3850 50  0001 C CNN
+	1    7000 3850
+	0    1    1    0
+$EndComp
 $EndSCHEMATC

Commit message: Finished esp8266 schematics
Parts:
- removed JP?: Jumper_2_Open, symbol Jumper:Jumper_2_Open
- removed R? (x3): 10K, symbol Device:R
- removed R?: 200R, symbol Device:R
- removed U?: W25Q16JVSSIQ, SOIC127P790X216-8N, symbol meteostation-rescue:W25Q16JVSSIQ-FLASH
- added AE?: Antenna_Chip, Connector_Coaxial:SMA_Molex_73251-2200_Horizontal, symbol Device:Antenna_Chip
- added C?: 10pF TBD, symbol Device:C
- added C?: 2.4pF TBD, symbol Device:C
- added C? (x2): 100nF, symbol Device:C
- added JP?: Jumper_PROG, symbol Jumper:Jumper_2_Open
- added JP?: Jumper_SPI_BOOT, symbol Jumper:Jumper_2_Bridged
- added L?: 1.6nH TBD, symbol Device:L
- added R? (x4): 10K, symbol Device:R
- added R?: 470R, symbol Device:R
- added R? (x4): 100R, symbol Device:R
- added R?: 499R, symbol Device:R
- added R?: 50R, symbol Device:R
- added U?: AT45DB041E-SSHN-B, Package_SO:SOIC-8_5.275x5.275mm_P1.27mm, symbol Memory_Flash:AT45DB161D-SU
- added U?: TXB0106PWR, Package_SO:TSSOP-16_4.4x5mm_P0.65mm, symbol TXB0106PWR:TXB0106PWR
Connections:
- net labels added: +5V, CLK, CS, HSPI_CLK, HSPI_CS, HSPI_MISO, HSPI_MOSI, MISO, MOSI, RXD, SPI_CLK, SPI_CS, SPI_MISO, SPI_MOSI, TXD
- net labels removed: MTCK, MTDI, MTDO, MTMS
- wire segments 59 -> 71
- no-connect marks 3 -> 2
Other:
- note added: "50R"
- note added: "Logical Level Shifter"
- moved on the sheet: R?
