File: hardware/esp8266.sch (KiCad schematic (older format))
At the start: 34 parts, among them U2 ESP8266EX, U3 AT25SF081-SHD-T, Y1 YSX321SL_26MHz_10ppm

Commit message: Finish adding footprints
Parts:
- AE1: footprint Connector_Coaxial:SMA_Molex_73251-2200_Horizontal -> RF_Antenna:Texas_SWRA117D_2.4GHz_Right
- C10, C11, C14, C15, C16, C17, C18, C9: footprint (none) -> Capacitor_SMD:C_0805_2012Metric
- C12, C13: footprint (none) -> Capacitor_SMD:C_1206_3216Metric
- JP1: footprint (none) -> Connector_PinHeader_2.54mm:PinHeader_1x02_P2.54mm_Vertical
- L1, L2: footprint (none) -> Inductor_SMD:L_0603_1608Metric
- R10, R11, R12, R13, R15, R16, R17, R18, R19, R20, R21, R22, R23, R7, R8, R9: footprint (none) -> Resistor_SMD:R_0805_2012Metric
- R14: value 499R -> 100R; footprint (none) -> Resistor_SMD:R_0805_2012Metric
- U3: footprint (none) -> Package_SO:SOIC-8_5.23x5.23mm_P1.27mm
Connections:
- net GND: now also AE1.2 (PCB_Trace); no longer AE1.1 (FEED)
- net at C14.2, L2.1: now also AE1.1 (FEED); no longer AE1.2 (PCB_Trace)
Other:
- moved on the sheet: AE1, R18, R19, R20, R21, R22, R23

Commit message: Power part 1/2 done
Parts:
- removed JP1: Jumper_PROG, Connector_PinHeader_2.54mm:PinHeader_1x02_P2.54mm_Vertical, symbol Jumper:Jumper_2_Open
- added JP1: Jumper_PROG, Jumper:SolderJumper-2_P1.3mm_Open_TrianglePad1.0x1.5mm, symbol Jumper:SolderJumper_2_Open
Connections:
- net GND: now also JP1.2 (B)
- net at R13.2, U2.15 (GPIO0): now also JP1.1 (A)
Changed lines of the file:
@@
-$EndComp
-$Comp
-L Jumper:Jumper_2_Open JP1
-U 1 1 603825B2
-P 7450 3500
-F 0 "JP1" V 7404 3598 50  0000 L CNN
-F 1 "Jumper_PROG" V 7495 3598 50  0000 L CNN
-F 2 "Connector_PinHeader_2.54mm:PinHeader_1x02_P2.54mm_Vertical" H 7450 3500 50  0001 C CNN
-F 3 "~" H 7450 3500 50  0001 C CNN
-	1    7450 3500
-	0    1    1    0
 $EndComp
 $Comp
@@
 L power:GND #PWR035
 U 1 1 60391528
-P 7450 3700
-F 0 "#PWR035" H 7450 3450 50  0001 C CNN
-F 1 "GND" H 7455 3527 50  0000 C CNN
-F 2 "" H 7450 3700 50  0001 C CNN
-F 3 "" H 7450 3700 50  0001 C CNN
-	1    7450 3700
+P 7450 3600
+F 0 "#PWR035" H 7450 3350 50  0001 C CNN
+F 1 "GND" H 7455 3427 50  0000 C CNN
+F 2 "" H 7450 3600 50  0001 C CNN
+F 3 "" H 7450 3600 50  0001 C CNN
+	1    7450 3600
 	1    0    0    -1
 $EndComp
@@
 Wire Wire Line
 	8450 5850 8800 5850
+$Comp
+L Jumper:SolderJumper_2_Open JP1
+U 1 1 608CC5E3
+P 7450 3450
+F 0 "JP1" V 7404 3518 50  0000 L CNN
+F 1 "Jumper_PROG" V 7495 3518 50  0000 L CNN
+F 2 "Jumper:SolderJumper-2_P1.3mm_Open_TrianglePad1.0x1.5mm" H 7450 3450 50  0001 C CNN
+F 3 "~" H 7450 3450 50  0001 C CNN
+	1    7450 3450
+	0    1    1    0
+$EndComp
 $EndSCHEMATC
