File: hardware/meteostation.sch (KiCad schematic (older format))
At the start: 12 parts

Commit message: Finished esp8266 schematics
Parts:
- SW?: value SW_MEC_5G -> RESET_BTN
Changed lines of the file:
@@
 P 7800 4650
 F 0 "SW?" H 7800 4935 50  0000 C CNN
-F 1 "SW_MEC_5G" H 7850 4850 50  0000 C CNN
+F 1 "RESET_BTN" H 7850 4850 50  0000 C CNN
 F 2 "" H 7800 4850 50  0001 C CNN
 F 3 "http://www.apem.com/int/index.php?controller=attachment&id_attachment=488" H 7800 4850 50  0001 C CNN
@@
 	6350 3250 6500 3250
 $Sheet
-S 8250 1850 650  500
+S 8300 1800 1100 550
 U 60322A2E
 F0 "ESP8266" 50
 F1 "esp8266.sch" 50
+F2 "CHIP_DISABLE" I L 8300 2200 50
+F3 "TX" O L 8300 1900 50
+F4 "RX" I L 8300 2000 50
+F5 "SPI_MISO" O R 9400 2000 50
+F6 "SPI_CLK" I R 9400 2100 50
+F7 "SPI_CS" I R 9400 2200 50
+F8 "SPI_MOSI" I R 9400 1900 50
 $EndSheet
 $EndSCHEMATC
