File: hardware/meteostation.kicad_pcb (KiCad board)
At the start: 2 copper layers, 80 x 33 mm, 172 parts, among them J1 PROG_Conn, J2 105450-0101, J3 PM_Sensor, J4 Anemometer, Q1 SI2302, SW1 RESET_BTN, SW2 Button, U1 STM32L432KBUx, U10 MC74VHC1G14, U12 HP203B, U13 MQ-2, U14 DHT11, U2 ESP8266EX, U3 AT25SF081-SHD-T, U4 FUSB302BMPX, U5 TLV75533PDBV, U6 BQ25895RTW, U7 TPD4E02B04DQA, U8 SX1278IMLTRT, U9 TPAS179-92LF, X1 YSO110TR_8MHz_10ppm, X2 YSO120TK_32.768KHz_10ppm, Y1 YSX321SL_26MHz_10ppm, Y2 YSX321SL_32.0MHz_10ppm

Commit message: Power part 1/2 done
Parts:
- added REF**: MountingHole_3.2mm_M3, MountingHole:MountingHole_3.2mm_M3, F.Cu at (130.8, 158.8)
- added REF**: MountingHole_3.2mm_M3, MountingHole:MountingHole_3.2mm_M3, F.Cu at (189.2, 158.8)
- JP1: footprint Connector_PinHeader_2.54mm:PinHeader_1x02_P2.54mm_Vertical -> Jumper:SolderJumper-2_P1.3mm_Open_TrianglePad1.0x1.5mm
- JP2: footprint Jumper:SolderJumper-2_P1.3mm_Open_TrianglePad1.0x1.5mm -> Jumper:SolderJumper-2_P1.3mm_Open_Pad1.0x1.5mm
- moved JP6 163.0 mm to (253.0, 94.2)
- moved D1 99.3 mm to (141.6, 135.3), turned to 90 degrees
- moved C28 93.0 mm to (150.0, 140.5), turned to 180 degrees
- moved L3 84.2 mm to (149.6, 143.9), turned to 270 degrees
- moved R35 83.9 mm to (149.2, 137.2), turned to 180 degrees
- moved C27 83.5 mm to (149.8, 134.4)
- moved C31 81.6 mm to (146.2, 148.2)
- moved JP3 81.2 mm to (163.2, 144.8), turned to 90 degrees
- moved C30 78.4 mm to (156.0, 142.0), turned to 90 degrees
- moved JP5 76.1 mm to (67.4, 96.9)
- moved R32 75.9 mm to (144.1, 135.3), turned to 270 degrees
- moved JP4 73.4 mm to (160.4, 144.8), turned to 90 degrees
- moved C29 72.2 mm to (153.5, 142.0), turned to 90 degrees
- moved R39 71.6 mm to (135.3, 151.1)
- moved C33 62.1 mm to (132.7, 148.0)
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Connections:
- U7 pad 10: Net-(U7-Pad10) -> /Power and USB/D-
- U7 pad 6: Net-(U7-Pad6) -> /Power and USB/CC2
- U7 pad 7: Net-(U7-Pad7) -> /Power and USB/CC1
- U7 pad 9: Net-(U7-Pad9) -> /Power and USB/D+
Routing:
- net +3V3: track 28.2 -> 70.0 mm
- net /Power and USB/ControlSelect: track 0.00 -> 31.5 mm, vias 0 -> 2
- net VBUS: track 28.9 -> 56.4 mm, vias 3 -> 6
- net /Power and USB/USB_PWR_D+: track 0.00 -> 25.6 mm, vias 0 -> 2
- net /Power and USB/USB_PWR_D-: track 0.00 -> 25.6 mm, vias 0 -> 2
- net Net-(BT1-Pad1): track 0.00 -> 25.1 mm
- net /Power and USB/D+: track 12.7 -> 30.6 mm
- net /Power and USB/D-: track 11.1 -> 28.3 mm
- net VCC: track 13.0 -> 30.1 mm
- net GND: track 63.4 -> 77.2 mm, vias 13 -> 20
- net Net-(C28-Pad1): track 0.00 -> 12.5 mm
- net /SDA: track 3.96 -> 15.2 mm, vias 0 -> 1
- net /SCL: track 6.45 -> 16.0 mm, vias 0 -> 1
- net /FUSB302_INT: track 8.94 -> 16.9 mm, vias 0 -> 1
- net /Power and USB/CC1: track 19.4 -> 23.9 mm, vias 0 -> 2
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Other:
- board size 80 x 33 mm -> 69.9 x 33 mm

Commit message: Finished power PCB part
Parts:
- moved D1 14.6 mm to (156.1, 134.4), turned to 270 degrees
- moved R29 11.1 mm to (138.8, 135.3), turned to 180 degrees
- moved R41 10.3 mm to (138.8, 144.8)
- moved R36 10.2 mm to (138.7, 141.4), turned to 180 degrees
- moved BT1 10.2 mm to (155.5, 155.4)
- moved TH1 10.2 mm to (145.3, 155.4)
- moved JP3 9.85 mm to (164.2, 135.0)
- moved JP4 9.82 mm to (161.0, 135.0)
- moved R30 8.70 mm to (135.1, 133.3), turned to 180 degrees
- moved R40 8.66 mm to (135.1, 140.1)
- moved D2 8.43 mm to (161.9, 144.4)
- moved C33 8.41 mm to (141.1, 147.3), turned to 180 degrees
- moved C34 8.30 mm to (163.6, 141.0)
- moved R28 7.55 mm to (135.1, 142.9), turned to 180 degrees
- moved C31 6.74 mm to (152.9, 148.0), turned to 90 degrees
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Connections:
- net /USB_DM renamed /USB_D-
- net /USB_DP renamed /USB_D+
- U7 pad 10: /Power and USB/D- -> Net-(U7-Pad10)
- U7 pad 6: /Power and USB/CC2 -> Net-(U7-Pad6)
- U7 pad 7: /Power and USB/CC1 -> Net-(U7-Pad7)
- U7 pad 9: /Power and USB/D+ -> Net-(U7-Pad9)
Routing:
- net +3V3: track 70.0 -> 136.4 mm, vias 2 -> 5
- net Net-(R41-Pad1): track 0.00 -> 63.0 mm, vias 0 -> 2
- net GND: track 77.2 -> 120.8 mm, vias 20 -> 26
- net VCC: track 30.1 -> 73.5 mm, vias 0 -> 2
- net VBUS: track 56.4 -> 93.7 mm, vias 6 -> 7
- net Net-(R39-Pad2): track 0.00 -> 35.0 mm, vias 0 -> 2
- net /Power and USB/D-: track 28.3 -> 53.0 mm, vias 2 -> 4
- net /Power and USB/D+: track 30.6 -> 55.3 mm, vias 2 -> 4
- net Net-(C33-Pad2): track 1.55 -> 19.6 mm, vias 1 -> 2
- net /SCL: track 16.0 -> 32.8 mm, vias 1 -> 2
- net /USB_D-: track 0.00 -> 16.5 mm
- net /USB_D+: track 0.00 -> 15.7 mm
- net /Charge: track 0.00 -> 14.8 mm, vias 0 -> 1
- net /BQ25895_INT: track 0.00 -> 13.7 mm, vias 0 -> 1
- net Net-(D1-Pad1): track 0.00 -> 12.9 mm
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Other:
- board size 69.9 x 33 mm -> 64.9 x 33 mm

Commit message: Finish esp8266 PCB part
Parts:
- added REF**: MountingHole_3.2mm_M3, MountingHole:MountingHole_3.2mm_M3, F.Cu at (112.3, 158.8)
- JP1: moved to B.Cu
- moved JP5 190.0 mm to (257.4, 94.0), turned to 180 degrees
- moved U3 90.3 mm to (121.9, 124.6), turned to 180 degrees
- moved C17 82.8 mm to (121.8, 110.3), turned to 270 degrees
- moved C18 81.9 mm to (116.0, 125.8), turned to 90 degrees
- moved AE1 76.4 mm to (112.2, 98.2)
- moved Y1 75.4 mm to (119.0, 111.8), turned to 270 degrees
- moved C13 74.7 mm to (119.0, 105.7)
- moved C12 73.8 mm to (123.8, 105.7)
- moved R11 73.7 mm to (124.9, 116.6), turned to 180 degrees
- moved R15 73.5 mm to (124.9, 114.5), turned to 180 degrees
- moved R9 72.3 mm to (118.9, 117.3), turned to 180 degrees
- moved R18 71.8 mm to (124.8, 120.6)
- moved R10 69.7 mm to (122.7, 118.6), turned to 180 degrees
- moved C16 69.5 mm to (121.8, 113.8), turned to 270 degrees
- moved C14 68.8 mm to (113.2, 99.9), turned to 180 degrees
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Connections:
- U7 pad 10: Net-(U7-Pad10) -> /Power and USB/D-
- U7 pad 6: Net-(U7-Pad6) -> /Power and USB/CC2
- U7 pad 7: Net-(U7-Pad7) -> /Power and USB/CC1
- U7 pad 9: Net-(U7-Pad9) -> /Power and USB/D+
Routing:
- net +3V3: track 136.4 -> 243.8 mm, vias 5 -> 13
- net GND: track 120.8 -> 145.6 mm, vias 26 -> 70
- net /ESP8266/HSPI_CLK: track 0.00 -> 21.4 mm
- net /ESP8266/CHIP_PU: track 0.00 -> 19.8 mm, vias 0 -> 3
- net Net-(R22-Pad1): track 0.00 -> 19.5 mm
- net /ESP8266/HSPI_MISO: track 0.00 -> 18.7 mm
- net /ESP8266/HSPI_MOSI: track 0.00 -> 15.1 mm
- net Net-(R23-Pad2): track 0.00 -> 13.9 mm, vias 0 -> 2
- net /ESP8266/RX: track 0.00 -> 13.4 mm, vias 0 -> 2
- net /ESP8266/HSPI_CS: track 0.00 -> 13.0 mm
- net Net-(R11-Pad2): track 0.00 -> 11.8 mm
- net Net-(R15-Pad2): track 0.00 -> 11.6 mm
- net Net-(R10-Pad2): track 0.00 -> 11.3 mm
- net Net-(R14-Pad2): track 0.00 -> 10.9 mm, vias 0 -> 2
- net Net-(C15-Pad2): track 0.00 -> 8.60 mm
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- added copper zone on F.Cu, net GND
Other:
- board size 64.9 x 33 mm -> 87.9 x 71.4 mm
